Commit message: Add files via upload

File: src/cart_description/urdf/invpend.urdf.xacro (robot description, xacro)
@@ -50,5 +50,5 @@
     <origin xyz="0 0 0" rpy="0 0 0"/>
     <axis xyz="1 0 0"/>
-    <limit effort="100.0" lower="-3.5" upper="3.5" velocity="10.0"/>
+    <limit effort="1000.0" lower="-3.5" upper="3.5" velocity="100.0"/>
     <dynamics damping="0.0"/>
     <transmission name="transmission_slider">
@@ -92,16 +92,6 @@
     <origin xyz="0 ${-depth/2-radius-radius_pole/2} ${height/4}" rpy="0 0 0"/>
     <axis xyz="0 1 0"/>
-    <limit effort="100.0" lower="${-PI}" upper = "${PI}" velocity="10.0"/>
+    <limit effort="100.0" lower="${-PI}" upper = "${PI}" velocity="100.0"/>
     <dynamics damping="0.0" friction="0.0"/>
-    <transmission name="transmission_pole">
-      <type>transmission_interface/SimpleTransmission</type>
-      <joint name="cart_to_pole">
-        <hardwareInterface>hardware_interface/EffortJointInterface</hardwareInterface>
-      </joint>
-      <actuator name="pole_motor">
-        <hardwareInterface>hardware_interface/EffortJointInterface</hardwareInterface>
-        <mechanicalReduction>1</mechanicalReduction>
-      </actuator>
-  </transmission>
   </joint>
   <!-- Pole Link -->

File: src/cart_description/urdf/ros2_control.xacro (robot description, xacro)
@@ -16,5 +16,4 @@
     </joint>
     <joint name="cart_to_pole">
-      <command_interface name="effort"/>
       <state_interface name="position"/>
          <param name="initial_value">0.0</param>

Commit message: working simulation of pympc

File: src/cart_description/urdf/invpend.urdf.xacro (robot description, xacro)
@@ -4,5 +4,5 @@
   <!-- Constants for robot dimensions -->
   <xacro:property name="PI" value="3.1415926535897931"/>
-  <xacro:property name="mass_slider" value="100" /> <!-- arbitrary value for mass -->
+  <xacro:property name="mass_slider" value="10" /> <!-- arbitrary value for mass -->
   <xacro:property name="mass_cart" value="20.0" /> <!-- arbitrary value for mass -->
   <xacro:property name="mass_pole" value="2.0" /> <!-- arbitrary value for mass -->
@@ -26,5 +26,4 @@
     <origin xyz="0 0 1"/>
   </joint>
-        <state_interface name="effort"/>
   <!-- Slider Link -->
   <link name="slidebar">
@@ -40,7 +39,7 @@
       <mass value="${mass_slider}"/>
       <inertia
-	  ixx="${mass_slider*length_slider*length_slider/12}" ixy="0.0" ixz="0.0"
-	  iyy="0.0" iyz="0.0"
-	  izz="${mass_slider*length_slider*length_slider/12}"/>
+	  ixx="${(1/12)*mass_slider*(radius*radius+radius*radius)}" ixy="0.0" ixz="0.0"
+	  iyy="${(1/12)*mass_slider*(length_slider*length_slider+radius*radius)}" iyz="0.0"
+	  izz="${(1/12)*mass_slider*(length_slider*length_slider+radius*radius)}"/>
     </inertial>
   </link>
@@ -50,6 +49,6 @@
     <origin xyz="0 0 0" rpy="0 0 0"/>
     <axis xyz="1 0 0"/>
-    <limit effort="1000.0" lower="-3.5" upper="3.5" velocity="100.0"/>
-    <dynamics damping="0.0"/>
+    <limit effort="100.0" lower="-3.5" upper="3.5" velocity="100.0"/>
+    <dynamics damping="0.0" friction="0.5"/>
     <transmission name="transmission_slider">
       <type>transmission_interface/SimpleTransmission</type>
@@ -82,7 +81,7 @@
       <mass value="${mass_cart}"/>
       <inertia
-	  ixx="${mass_cart*(depth*depth+height*height)/12}" ixy="0.0" ixz="0.0"
-	  iyy="${mass_cart*(depth*depth+width*width)/12}" iyz="0.0"
-	  izz="${mass_cart*(width*width+height*height)/12}"/>
+	  ixx="${(1/12)*mass_cart*(depth*depth+height*height)}" ixy="0.0" ixz="0.0"
+	  iyy="${(1/12)*mass_cart*(width*width+height*height)}" iyz="0.0"
+	  izz="${(1/12)*mass_cart*(width*width+depth*depth)}"/>
     </inertial>
   </link>
@@ -114,7 +113,7 @@
       <mass value="${mass_pole}"/>
       <inertia
-	  ixx="${mass_pole*(radius_pole*radius_pole+length_pole*length_pole)/12}" ixy="0.0" ixz="0.0"
-	  iyy="${mass_pole*(radius_pole*radius_pole+radius_pole*radius_pole)/12}" iyz="0.0"
-	  izz="${mass_pole*(radius_pole*radius_pole+length_pole*length_pole)/12}"/>
+	  ixx="${(1/12)*mass_pole*(radius_pole*radius_pole+length_pole*length_pole)}" ixy="0.0" ixz="0.0"
+	  iyy="${(1/12)*mass_pole*(radius_pole*radius_pole+length_pole*length_pole)}" iyz="0.0"
+	  izz="${(1/12)*mass_pole*(radius_pole*radius_pole+radius_pole*radius_pole)}"/>
     </inertial>
   </link>

File: src/cart_description/urdf/ros2_control.xacro (robot description, xacro)
@@ -7,6 +7,6 @@
     <joint name= "slider_to_cart">
         <command_interface name="effort">
-          <param name="min">-1000</param>
-          <param name="max">1000</param>
+          <param name="min">-10</param>
+          <param name="max">10</param>
         </command_interface>
         <state_interface name="position">
@@ -17,5 +17,5 @@
     <joint name="cart_to_pole">
       <state_interface name="position"/>
-         <param name="initial_value">0.0</param>
+         <param name="initial_value">1.57</param>
       <state_interface name="velocity"/>
     </joint>
